File: VdpBooster/VdpBooster.kicad_sch (KiCad schematic)
At the start: 30 parts, among them U1 M5M4C264L, U2 M5M4C264L, U3 M5M4C264L, U4 M5M4C264L, U5 315-5313A

Commit message: v101 changes
Parts:
- C6: renamed from C1; now not fitted; now left out of the parts list
- C7: renamed from C2; now not fitted; now left out of the parts list
- C8: renamed from C3; now not fitted; now left out of the parts list
- C9: renamed from C4; now not fitted; now left out of the parts list
- renumbered C6 to C1, C7 to C2, C8 to C3, C5 to C4, C9 to C5
Changed lines of the file:
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@@
 		(body_style 1)
 		(exclude_from_sim no)
-		(in_bom yes)
-		(on_board yes)
-		(in_pos_files yes)
-		(dnp no)
+		(in_bom no)
+		(on_board no)
+		(in_pos_files no)
+		(dnp yes)
 		(fields_autoplaced yes)
-		(property "Reference" "C2"
+		(property "Reference" "C7"
 			(at 250.19 121.9199 0)
 			(show_name no)
@@
 			(project "VdpBooster"
 				(path "/5c12a977-b9b7-4efa-87b3-dae48c707533"
-					(reference "C2")
+					(reference "C7")
 					(unit 1)
 				)
@@
 		(body_style 1)
 		(exclude_from_sim no)
-		(in_bom yes)
-		(on_board yes)
-		(in_pos_files yes)
-		(dnp no)
+		(in_bom no)
+		(on_board no)
+		(in_pos_files no)
+		(dnp yes)
 		(fields_autoplaced yes)
-		(property "Reference" "C4"
+		(property "Reference" "C9"
 			(at 275.59 121.9199 0)
 			(show_name no)
@@
 			(project "VdpBooster"
 				(path "/5c12a977-b9b7-4efa-87b3-dae48c707533"
-					(reference "C4")
+					(reference "C9")
 					(unit 1)
 				)
@@
 		(body_style 1)
 		(exclude_from_sim no)
-		(in_bom yes)
-		(on_board yes)
-		(in_pos_files yes)
-		(dnp no)
+		(in_bom no)
+		(on_board no)
+		(in_pos_files no)
+		(dnp yes)
 		(fields_autoplaced yes)
-		(property "Reference" "C3"
+		(property "Reference" "C8"
 			(at 262.89 121.9199 0)
 			(show_name no)
@@
 			(project "VdpBooster"
 				(path "/5c12a977-b9b7-4efa-87b3-dae48c707533"
-					(reference "C3")
+					(reference "C8")
 					(unit 1)
 				)
@@
 		(dnp no)
 		(fields_autoplaced yes)
-		(property "Reference" "C7"
+		(property "Reference" "C2"
 			(at 173.99 157.48 90)
 			(show_name no)
@@
 			(project "VdpBooster"
 				(path "/5c12a977-b9b7-4efa-87b3-dae48c707533"
-					(reference "C7")
+					(reference "C2")
 					(unit 1)
 				)
@@
 		(body_style 1)
 		(exclude_from_sim no)
-		(in_bom yes)
-		(on_board yes)
-		(in_pos_files yes)
-		(dnp no)
+		(in_bom no)
+		(on_board no)
+		(in_pos_files no)
+		(dnp yes)
 		(fields_autoplaced yes)
-		(property "Reference" "C1"
+		(property "Reference" "C6"
 			(at 236.22 121.9199 0)
 			(show_name no)
@@
 			(project "VdpBooster"
 				(path "/5c12a977-b9b7-4efa-87b3-dae48c707533"
-					(reference "C1")
+					(reference "C6")
 					(unit 1)
 				)
@@
 		(in_pos_files yes)
 		(dnp no)
-		(property "Reference" "C5"
+		(property "Reference" "C4"
 			(at 19.05 160.0199 0)
 			(show_name no)
@@
 			(project "VdpBooster"
 				(path "/5c12a977-b9b7-4efa-87b3-dae48c707533"
-					(reference "C5")
+					(reference "C4")
 					(unit 1)
 				)
@@
 		(dnp no)
 		(fields_autoplaced yes)
-		(property "Reference" "C8"
+		(property "Reference" "C3"
 			(at 173.99 182.88 90)
 			(show_name no)
@@
 			(project "VdpBooster"
 				(path "/5c12a977-b9b7-4efa-87b3-dae48c707533"
-					(reference "C8")
+					(reference "C3")
 					(unit 1)
 				)
@@
 		(dnp no)
 		(fields_autoplaced yes)
-		(property "Reference" "C6"
+		(property "Reference" "C1"
 			(at 173.99 132.08 90)
 			(show_name no)
@@
 			(project "VdpBooster"
 				(path "/5c12a977-b9b7-4efa-87b3-dae48c707533"
-					(reference "C6")
+					(reference "C1")
 					(unit 1)
 				)
@@
 		(dnp no)
 		(fields_autoplaced yes)
-		(property "Reference" "C9"
+		(property "Reference" "C5"
 			(at 130.81 157.4799 0)
 			(show_name no)
@@
 			(project "VdpBooster"
 				(path "/5c12a977-b9b7-4efa-87b3-dae48c707533"
-					(reference "C9")
+					(reference "C5")
 					(unit 1)
 				)
